File: KiCad/SCART_Cable_Breakout.kicad_sch (KiCad schematic)
At the start: 17 parts, among them J1 SCART-F, J2 SCART Cable, U1 ST662A

Commit message: Edit silkscreen labels.
Parts:
- C1, C2, C3: value 220 uF -> 220uF
Changed lines of the file:
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@@
 			)
 		)
-		(property "Value" "220 uF"
+		(property "Value" "220uF"
 			(at 161.29 47.498 90)
 			(effects
@@
 			)
 		)
-		(property "Value" "220 uF"
+		(property "Value" "220uF"
 			(at 161.29 75.438 90)
 			(effects
@@
 			)
 		)
-		(property "Value" "220 uF"
+		(property "Value" "220uF"
 			(at 161.29 61.468 90)
 			(effects

Commit message: Change PCB outline to match more common SCART connectors. Remove solder jumpers for RGB capacitors. 5V->12V converter: replace electrolytic capacitors with size B tantalum ones.
Parts:
- removed JP1, JP2, JP3: SolderJumper_2_Open, Jumper:SolderJumper-2_P1.3mm_Open_RoundedPad1.0x1.5mm, symbol Jumper:SolderJumper_2_Open
- C7, C8: footprint Capacitor_SMD:CP_Elec_6.3x3.9 -> Capacitor_Tantalum_SMD:CP_EIA-3528-21_Kemet-B_Pad1.50x2.35mm_HandSolder
